Commit message: Add laser scanner

File: urdf/m2wr.xacro (robot description, xacro)
@@ -61,4 +61,31 @@
     </visual>
     </link>
+<!-- Laser scanner  -->
+<link name="sensor_laser">
+    <inertial>
+      <origin xyz="0 0 0" rpy="0 0 0" />
+      <mass value="1" />
+      <!-- RANDOM INERTIA BELOW -->
+      <xacro:cylinder_inertia mass="1" r="0.05" l="0.1" />
+    </inertial>
+    <visual>
+      <origin xyz="0 0 0" rpy="0 0 0" />
+      <geometry>
+        <cylinder radius="0.05" length="0.1"/>
+      </geometry>
+      <material name="white" />
+    </visual>
+    <collision>
+      <origin xyz="0 0 0" rpy="0 0 0"/>
+      <geometry>
+        <cylinder radius="0.05" length="0.1"/>
+      </geometry>
+    </collision>
+  </link>
+  <joint name="joint_sensor_laser" type="fixed">
+    <origin xyz="0.15 0 0.05" rpy="0 0 0"/>
+    <parent link="link_chassis"/>
+    <child link="sensor_laser"/>
+  </joint>
   <!-- Create wheel right -->
     <xacro:link_wheel name="link_right_wheel"/>

File: urdf/macro.xacro (robot description, xacro)
@@ -32,3 +32,7 @@
       </joint>
     </xacro:macro>
+    <!-- Laser scanner -->
+    <xacro:macro name="cylinder_inertia" params="mass r l">
+      <inertia ixx="${mass*(3*r*r+l*l)/12}" ixy = "0" ixz = "0" iyy="${mass*(3*r*r+l*l)/12}" iyz = "0" izz="${mass*(r*r)/2}" />
+    </xacro:macro>
 </robot>

Commit message: Minor fixes

File: urdf/m2wr.xacro (robot description, xacro)
@@ -60,7 +60,7 @@
       </geometry>
     </visual>
-    </link>
-<!-- Laser scanner  -->
-<link name="sensor_laser">
+  </link>
+  <!-- Laser scanner  -->
+  <link name="sensor_laser">
     <inertial>
       <origin xyz="0 0 0" rpy="0 0 0" />
@@ -88,11 +88,8 @@
     <child link="sensor_laser"/>
   </joint>
-  <!-- Create wheel right -->
-    <xacro:link_wheel name="link_right_wheel"/>
-  <!--   Joint for right wheel  -->
-    <xacro:joint_wheel name="joint_right_wheel" child="link_right_wheel" origin_xyz="-0.05 0.15 0"/>
-  <!-- Left Wheel link -->
+  <!-- Create wheels -->
+  <xacro:link_wheel name="link_right_wheel"/>
+  <xacro:joint_wheel name="joint_right_wheel" child="link_right_wheel" origin_xyz="-0.05 0.15 0"/>
   <xacro:link_wheel name="link_left_wheel"/>
-   <!--   Joint for right wheel  -->
   <xacro:joint_wheel name="joint_left_wheel" child="link_left_wheel" origin_xyz="-0.05 -0.15 0"/>
  </robot>

File: urdf/macro.xacro (robot description, xacro)
@@ -8,5 +8,6 @@
                 <inertia ixx="0.000526666666667" ixy="0" ixz="0" iyy="0.000526666666667" iyz="0" izz="0.001"/>
             </inertial>
-            <collision name="link_right_wheel_collision">
+            <!-- <collision name="link_right_wheel_collision"> -->
+            <collision name="${name}_collision">
               <origin rpy="0 1.5707 1.5707" xyz="0 0 0"/>
               <geometry>

Commit message: M2WR-14: Minor changes

File: urdf/m2wr.xacro (robot description, xacro)
@@ -4,92 +4,79 @@
     <xacro:include filename="$(find mtracker)/urdf/m2wr.gazebo"/>
     <xacro:include filename="$(find mtracker)/urdf/macro.xacro"/>
-  <link name="link_chassis">
-    <!-- pose and inertial -->
-    <pose>0 0 0.1 0 0 0</pose>
-    <inertial>
-      <mass value="5"/>
-      <origin rpy="0 0 0" xyz="0 0 0.1"/>
-      <inertia ixx="0.0395416666667" ixy="0" ixz="0" iyy="0.106208333333" iyz="0" izz="0.106208333333"/>
-    </inertial>
-    <collision name="collision_chassis">
-      <geometry>
-        <box size="0.5 0.3 0.07"/>
-      </geometry>
-    </collision>
-    <visual>
-      <origin rpy="0 0 0" xyz="0 0 0"/>
-      <geometry>
-        <box size="0.5 0.3 0.07"/>
-      </geometry>
-      <material name="blue"/>
-    </visual>
-    <!-- Mtracker dimensions  -->
-  <!-- <collision name="collision_chassis">
-      <geometry>
-        <cylinder length="0.3" radius="0.05"/>
-      </geometry>
-  </collision>
-    <visual>
-      <origin rpy="0 0 0" xyz="0 0 0"/>
-      <geometry>
-        <cylinder length="0.3" radius="0.05"/>
-      </geometry>
-      <material name="blue"/>
-    </visual>  -->
-    <!-- caster front -->
-    <collision name="caster_front_collision">
-      <origin rpy=" 0 0 0" xyz="0.35 0 -0.05"/>
-      <geometry>
-        <sphere radius="0.05"/>
-      </geometry>
-      <surface>
-        <friction>
-          <ode>
-            <mu>0</mu>
-            <mu2>0</mu2>
-            <slip1>1.0</slip1>
-            <slip2>1.0</slip2>
-          </ode>
-        </friction>
-      </surface>
-    </collision>
-    <visual name="caster_front_visual">
-      <origin rpy=" 0 0 0" xyz="0.2 0 -0.05"/>
-      <geometry>
-        <sphere radius="0.05"/>
-      </geometry>
-    </visual>
-  </link>
-  <!-- Laser scanner  -->
-  <link name="sensor_laser">
-    <inertial>
-      <origin xyz="0 0 0" rpy="0 0 0" />
-      <mass value="1" />
-      <!-- RANDOM INERTIA BELOW -->
-      <xacro:cylinder_inertia mass="1" r="0.05" l="0.1" />
-    </inertial>
-    <visual>
-      <origin xyz="0 0 0" rpy="0 0 0" />
-      <geometry>
-        <cylinder radius="0.05" length="0.1"/>
-      </geometry>
-      <material name="white" />
-    </visual>
-    <collision>
-      <origin xyz="0 0 0" rpy="0 0 0"/>
-      <geometry>
-        <cylinder radius="0.05" length="0.1"/>
-      </geometry>
-    </collision>
-  </link>
-  <joint name="joint_sensor_laser" type="fixed">
-    <origin xyz="0.15 0 0.05" rpy="0 0 0"/>
-    <parent link="link_chassis"/>
-    <child link="sensor_laser"/>
-  </joint>
-  <!-- Create wheels -->
-  <xacro:link_wheel name="link_right_wheel"/>
-  <xacro:joint_wheel name="joint_right_wheel" child="link_right_wheel" origin_xyz="-0.05 0.15 0"/>
-  <xacro:link_wheel name="link_left_wheel"/>
-  <xacro:joint_wheel name="joint_left_wheel" child="link_left_wheel" origin_xyz="-0.05 -0.15 0"/>
- </robot>
+    <link name="link_chassis">
+        <!-- pose and inertial -->
+        <pose>0 0 0.1 0 0 0</pose>
+        <inertial>
+            <mass value="5"/>
+            <origin rpy="0 0 0" xyz="0 0 0.1"/>
+            <inertia ixx="0.0395416666667" ixy="0" ixz="0" iyy="0.106208333333" iyz="0" izz="0.106208333333"/>
+        </inertial>
+        <collision name="collision_chassis">
+            <geometry>
+                <box size="0.5 0.3 0.07"/>
+            </geometry>
+        </collision>
+        <visual>
+            <origin rpy="0 0 0" xyz="0 0 0"/>
+            <geometry>
+                <box size="0.5 0.3 0.07"/>
+            </geometry>
+            <material name="blue"/>
+        </visual>
+        <!-- caster front -->
+        <collision name="caster_front_collision">
+            <origin rpy=" 0 0 0" xyz="0.35 0 -0.05"/>
+            <geometry>
+                <sphere radius="0.05"/>
+            </geometry>
+            <surface>
+                <friction>
+                    <ode>
+                        <mu>0</mu>
+                        <mu2>0</mu2>
+                        <slip1>1.0</slip1>
+                        <slip2>1.0</slip2>
+                    </ode>
+                </friction>
+            </surface>
+        </collision>
+        <visual name="caster_front_visual">
+            <origin rpy=" 0 0 0" xyz="0.2 0 -0.05"/>
+            <geometry>
+                <sphere radius="0.05"/>
+            </geometry>
+        </visual>
+    </link>
+    <!-- Laser scanner  -->
+    <link name="sensor_laser">
+        <inertial>
+            <origin xyz="0 0 0" rpy="0 0 0" />
+            <mass value="1" />
+                <!-- RANDOM INERTIA BELOW -->
+            <xacro:cylinder_inertia mass="1" r="0.05" l="0.1" />
+        </inertial>
+        <visual>
+            <origin xyz="0 0 0" rpy="0 0 0" />
+            <geometry>
+                <cylinder radius="0.05" length="0.1"/>
+            </geometry>
+            <material name="white" />
+        </visual>
+        <collision>
+            <origin xyz="0 0 0" rpy="0 0 0"/>
+            <geometry>
+                <cylinder radius="0.05" length="0.1"/>
+            </geometry>
+        </collision>
+    </link>
+    <joint name="joint_sensor_laser" type="fixed">
+        <origin xyz="0.15 0 0.05" rpy="0 0 0"/>
+        <parent link="link_chassis"/>
+        <child link="sensor_laser"/>
+    </joint>
+    <!-- Create wheels -->
+    <xacro:link_wheel name="link_right_wheel"/>
+    <xacro:joint_wheel name="joint_right_wheel" child="link_right_wheel" origin_xyz="-0.05 0.15 0"/>
+    <xacro:link_wheel name="link_left_wheel"/>
+    <xacro:joint_wheel name="joint_left_wheel" child="link_left_wheel" origin_xyz="-0.05 -0.15 0"/>
+</robot>

Commit message: M2WR-14: Update diff drive controller, add minor changes

File: urdf/m2wr.xacro (robot description, xacro)
@@ -12,4 +12,5 @@
             <inertia ixx="0.0395416666667" ixy="0" ixz="0" iyy="0.106208333333" iyz="0" izz="0.106208333333"/>
         </inertial>
+        <!-- body -->
         <collision name="collision_chassis">
             <geometry>
@@ -48,14 +49,12 @@
         </visual>
     </link>
-    <!-- Laser scanner  -->
     <link name="sensor_laser">
         <inertial>
-            <origin xyz="0 0 0" rpy="0 0 0" />
+            <origin xyz="0 0 0" rpy="0 0 0"/>
             <mass value="1" />
-                <!-- RANDOM INERTIA BELOW -->
             <xacro:cylinder_inertia mass="1" r="0.05" l="0.1" />
         </inertial>
         <visual>
-            <origin xyz="0 0 0" rpy="0 0 0" />
+            <origin xyz="0 0 0" rpy="0 0 0"/>
             <geometry>
                 <cylinder radius="0.05" length="0.1"/>
@@ -77,6 +76,6 @@
     <!-- Create wheels -->
     <xacro:link_wheel name="link_right_wheel"/>
-    <xacro:joint_wheel name="joint_right_wheel" child="link_right_wheel" origin_xyz="-0.05 0.15 0"/>
+    <xacro:joint_wheel name="joint_right_wheel" child="link_right_wheel" origin_xyz="-0.05 0.20 0"/>
     <xacro:link_wheel name="link_left_wheel"/>
-    <xacro:joint_wheel name="joint_left_wheel" child="link_left_wheel" origin_xyz="-0.05 -0.15 0"/>
+    <xacro:joint_wheel name="joint_left_wheel" child="link_left_wheel" origin_xyz="-0.05 -0.20 0"/>
 </robot>

File: urdf/macro.xacro (robot description, xacro)
@@ -8,6 +8,6 @@
                 <inertia ixx="0.000526666666667" ixy="0" ixz="0" iyy="0.000526666666667" iyz="0" izz="0.001"/>
             </inertial>
-            <!-- <collision name="link_right_wheel_collision"> -->
-            <collision name="${name}_collision">
+            <collision name="link_right_wheel_collision">
+            <!-- <collision name="${name}_collision"> -->
               <origin rpy="0 1.5707 1.5707" xyz="0 0 0"/>
               <geometry>
@@ -35,5 +35,7 @@
     <!-- Laser scanner -->
     <xacro:macro name="cylinder_inertia" params="mass r l">
-      <inertia ixx="${mass*(3*r*r+l*l)/12}" ixy = "0" ixz = "0" iyy="${mass*(3*r*r+l*l)/12}" iyz = "0" izz="${mass*(r*r)/2}" />
+      <inertia ixx="${mass*(3*r*r+l*l)/12}" ixy = "0" ixz = "0"
+               iyy="${mass*(3*r*r+l*l)/12}" iyz = "0"
+               izz="${mass*(r*r)/2}"/>
     </xacro:macro>
 </robot>

Commit message: M2WR-15: Code cleanup, add RViz to launchfile

File: urdf/m2wr.xacro (robot description, xacro)
@@ -34,6 +34,6 @@
                 <friction>
                     <ode>
-                        <mu>0</mu>
-                        <mu2>0</mu2>
+                        <mu>0.1</mu>
+                        <mu2>0.1</mu2>
                         <slip1>1.0</slip1>
                         <slip2>1.0</slip2>
@@ -76,6 +76,6 @@
     <!-- Create wheels -->
     <xacro:link_wheel name="link_right_wheel"/>
-    <xacro:joint_wheel name="joint_right_wheel" child="link_right_wheel" origin_xyz="-0.05 0.20 0"/>
+    <xacro:joint_wheel name="joint_right_wheel" child="link_right_wheel" origin_xyz="-0.05 0.15 0"/>
     <xacro:link_wheel name="link_left_wheel"/>
-    <xacro:joint_wheel name="joint_left_wheel" child="link_left_wheel" origin_xyz="-0.05 -0.20 0"/>
+    <xacro:joint_wheel name="joint_left_wheel" child="link_left_wheel" origin_xyz="-0.05 -0.15 0"/>
 </robot>

File: urdf/macro.xacro (robot description, xacro)
@@ -28,5 +28,6 @@
         <child link="${child}"/>
         <parent link="link_chassis"/>
-        <axis rpy="0 0 0" xyz="0 1 0"/>
+        <!-- <axis rpy="0 0 0" xyz="0 1 0"/> -->
+        <axis xyz="0 1 0"/>
         <limit effort="10000" velocity="1000"/>
         <joint_properties damping="1.0" friction="1.0"/>

Commit message: M2WR-7: Robot now drives properly

File: urdf/m2wr.xacro (robot description, xacro)
@@ -6,8 +6,8 @@
     <link name="link_chassis">
         <!-- pose and inertial -->
-        <pose>0 0 0.1 0 0 0</pose>
+        <pose>0 0 0.01 0 0 0</pose>
         <inertial>
-            <mass value="5"/>
-            <origin rpy="0 0 0" xyz="0 0 0.1"/>
+            <mass value="1.8"/>
+            <origin rpy="0 0 0" xyz="0 0 0.01"/>
             <inertia ixx="0.0395416666667" ixy="0" ixz="0" iyy="0.106208333333" iyz="0" izz="0.106208333333"/>
         </inertial>
@@ -15,11 +15,27 @@
         <collision name="collision_chassis">
             <geometry>
-                <box size="0.5 0.3 0.07"/>
+                <cylinder length="0.045" radius="0.084"/>
             </geometry>
         </collision>
         <visual>
-            <origin rpy="0 0 0" xyz="0 0 0"/>
+            <origin rpy="0 0 0" xyz="0 0 0.010"/>
             <geometry>
-                <box size="0.5 0.3 0.07"/>
+                <cylinder length="0.045" radius="0.084"/>
+            </geometry>
+            <material name="blue"/>
+        </visual>
+        <!-- controller -->
+        <visual>
+            <origin rpy="0 0 0" xyz="0 0 0.046"/>
+            <geometry>
+                <cylinder length="0.025" radius="0.080"/>
+            </geometry>
+            <material name="blue"/>
+        </visual>
+        <!-- intel nuc -->
+        <visual>
+            <origin rpy="0 0 0" xyz="0 0 0.071"/>
+            <geometry>
+                <box size="0.1 0.1 0.06"/>
             </geometry>
             <material name="blue"/>
@@ -27,7 +43,7 @@
         <!-- caster front -->
         <collision name="caster_front_collision">
-            <origin rpy=" 0 0 0" xyz="0.35 0 -0.05"/>
+            <origin rpy="0 0 0" xyz="0.08 0 -0.015"/>
             <geometry>
-                <sphere radius="0.05"/>
+                <cylinder length="0.01" radius="0.003"/>
             </geometry>
             <surface>
@@ -43,15 +59,53 @@
         </collision>
         <visual name="caster_front_visual">
-            <origin rpy=" 0 0 0" xyz="0.2 0 -0.05"/>
+            <origin rpy="0 0 0" xyz="0.08 0 -0.015"/>
             <geometry>
-                <sphere radius="0.05"/>
+                <cylinder length="0.01" radius="0.003"/>
+            </geometry>
+        </visual>
+        <!-- caster back -->
+        <collision name="caster_back_collision">
+            <origin rpy="0 0 0" xyz="-0.08 0 -0.015"/>
+            <geometry>
+                <cylinder length="0.01" radius="0.003"/>
+            </geometry>
+            <surface>
+                <friction>
+                    <ode>
+                        <mu>0.1</mu>
+                        <mu2>0.1</mu2>
+                        <slip1>1.0</slip1>
+                        <slip2>1.0</slip2>
+                    </ode>
+                </friction>
+            </surface>
+        </collision>
+        <visual name="caster_back_visual">
+            <origin rpy="0 0 0" xyz="-0.08 0 -0.015"/>
+            <geometry>
+                <cylinder length="0.01" radius="0.003"/>
             </geometry>
         </visual>
     </link>
-    <link name="sensor_laser">
+    <!-- simple line to indicate front -->
+    <link name="front_indicator">
+        <parent link="link_chassis"/>
+        <visual>
+            <origin rpy="0 0 0" xyz="0.05 0 0"/>
+            <geometry>
+                <box size="0.045 0.005 0.001"/>
+            </geometry>
+        </visual>
+    </link>
+    <joint name="front_indicatior_joint" type="fixed">
+        <parent link="link_chassis"/>
+        <child link="front_indicator"/>
+        <origin rpy="0 0 0" xyz="0 0 0.071"/>
+    </joint>
+    <!-- <link name="sensor_laser">
         <inertial>
             <origin xyz="0 0 0" rpy="0 0 0"/>
-            <mass value="1" />
-            <xacro:cylinder_inertia mass="1" r="0.05" l="0.1" />
+            <mass value="0.1" />
+            <xacro:cylinder_inertia mass="0.1" r="0.05" l="0.1" />
         </inertial>
         <visual>
@@ -73,9 +127,9 @@
         <parent link="link_chassis"/>
         <child link="sensor_laser"/>
-    </joint>
+    </joint> -->
     <!-- Create wheels -->
     <xacro:link_wheel name="link_right_wheel"/>
-    <xacro:joint_wheel name="joint_right_wheel" child="link_right_wheel" origin_xyz="-0.05 0.15 0"/>
+    <xacro:joint_wheel name="joint_right_wheel" child="link_right_wheel" origin_xyz="0 0.075 0"/>
     <xacro:link_wheel name="link_left_wheel"/>
-    <xacro:joint_wheel name="joint_left_wheel" child="link_left_wheel" origin_xyz="-0.05 -0.15 0"/>
+    <xacro:joint_wheel name="joint_left_wheel" child="link_left_wheel" origin_xyz="0 -0.075 0"/>
 </robot>

File: urdf/macro.xacro (robot description, xacro)
@@ -4,13 +4,12 @@
         <link name="${name}">
             <inertial>
-                <mass value="0.2"/>
+                <mass value="0.1"/>
                 <origin rpy="0 1.5707 1.5707" xyz="0 0 0"/>
                 <inertia ixx="0.000526666666667" ixy="0" ixz="0" iyy="0.000526666666667" iyz="0" izz="0.001"/>
             </inertial>
-            <collision name="link_right_wheel_collision">
-            <!-- <collision name="${name}_collision"> -->
+            <collision name="${name}_collision">
               <origin rpy="0 1.5707 1.5707" xyz="0 0 0"/>
               <geometry>
-                <cylinder length="0.04" radius="0.1"/>
+                <cylinder length="0.003" radius="0.026"/>
               </geometry>
             </collision>
@@ -18,5 +17,5 @@
               <origin rpy="0 1.5707 1.5707" xyz="0 0 0"/>
               <geometry>
-                <cylinder length="0.04" radius="0.1"/>
+                <cylinder length="0.003" radius="0.026"/>
               </geometry>
             </visual>
@@ -35,8 +34,8 @@
     </xacro:macro>
     <!-- Laser scanner -->
-    <xacro:macro name="cylinder_inertia" params="mass r l">
+    <!-- <xacro:macro name="cylinder_inertia" params="mass r l">
       <inertia ixx="${mass*(3*r*r+l*l)/12}" ixy = "0" ixz = "0"
                iyy="${mass*(3*r*r+l*l)/12}" iyz = "0"
                izz="${mass*(r*r)/2}"/>
-    </xacro:macro>
+    </xacro:macro> -->
 </robot>
