Commit message: refactor: just some minor changes

File: urdf/m2wr.xacro (robot description, xacro)
@@ -1,49 +1,52 @@
 <?xml version="1.0"?>
 <robot name="mtracker" xmlns:xacro="https://www.ros.org/wiki/xacro">
-    <xacro:include filename="$(find mtracker)/urdf/materials.xacro"/>
-    <xacro:include filename="$(find mtracker)/urdf/m2wr.gazebo"/>
-    <xacro:include filename="$(find mtracker)/urdf/macro.xacro"/>
+    <xacro:include filename="$(find mtracker)/urdf/materials.xacro" />
+    <xacro:include filename="$(find mtracker)/urdf/m2wr.gazebo" />
+    <xacro:include filename="$(find mtracker)/urdf/macro.xacro" />
+    <link name="dummy">
+        <pose>0 0 0 0 0 0</pose>
+    </link>
     <link name="link_chassis">
         <!-- pose and inertial -->
         <pose>0 0 0.01 0 0 0</pose>
         <inertial>
-            <mass value="1.8"/>
-            <origin rpy="0 0 0" xyz="0 0 0.01"/>
-            <inertia ixx="0.0395416666667" ixy="0" ixz="0" iyy="0.106208333333" iyz="0" izz="0.106208333333"/>
+            <mass value="1.8" />
+            <origin rpy="0 0 0" xyz="0 0 0.01" />
+            <inertia ixx="0.0395416666667" ixy="0" ixz="0" iyy="0.106208333333" iyz="0" izz="0.106208333333" />
         </inertial>
         <!-- body -->
         <collision name="collision_chassis">
             <geometry>
-                <cylinder length="0.045" radius="0.084"/>
+                <cylinder length="0.045" radius="0.084" />
             </geometry>
         </collision>
         <visual>
-            <origin rpy="0 0 0" xyz="0 0 0.010"/>
+            <origin rpy="0 0 0" xyz="0 0 0.010" />
             <geometry>
-                <cylinder length="0.045" radius="0.084"/>
+                <cylinder length="0.045" radius="0.084" />
             </geometry>
-            <material name="blue"/>
+            <material name="blue" />
         </visual>
         <!-- controller -->
         <visual>
-            <origin rpy="0 0 0" xyz="0 0 0.046"/>
+            <origin rpy="0 0 0" xyz="0 0 0.046" />
             <geometry>
-                <cylinder length="0.025" radius="0.080"/>
+                <cylinder length="0.025" radius="0.080" />
             </geometry>
-            <material name="blue"/>
+            <material name="blue" />
         </visual>
         <!-- intel nuc -->
         <visual>
-            <origin rpy="0 0 0" xyz="0 0 0.071"/>
+            <origin rpy="0 0 0" xyz="0 0 0.071" />
             <geometry>
-                <box size="0.1 0.1 0.06"/>
+                <box size="0.1 0.1 0.06" />
             </geometry>
-            <material name="blue"/>
+            <material name="blue" />
         </visual>
         <!-- caster front -->
         <collision name="caster_front_collision">
-            <origin rpy="0 0 0" xyz="0.08 0 -0.015"/>
+            <origin rpy="0 0 0" xyz="0.08 0 -0.015" />
             <geometry>
-                <cylinder length="0.01" radius="0.003"/>
+                <cylinder length="0.01" radius="0.003" />
             </geometry>
             <surface>
@@ -59,14 +62,14 @@
         </collision>
         <visual name="caster_front_visual">
-            <origin rpy="0 0 0" xyz="0.08 0 -0.015"/>
+            <origin rpy="0 0 0" xyz="0.08 0 -0.015" />
             <geometry>
-                <cylinder length="0.01" radius="0.003"/>
+                <cylinder length="0.01" radius="0.003" />
             </geometry>
         </visual>
         <!-- caster back -->
         <collision name="caster_back_collision">
-            <origin rpy="0 0 0" xyz="-0.08 0 -0.015"/>
+            <origin rpy="0 0 0" xyz="-0.08 0 -0.015" />
             <geometry>
-                <cylinder length="0.01" radius="0.003"/>
+                <cylinder length="0.01" radius="0.003" />
             </geometry>
             <surface>
@@ -82,24 +85,29 @@
         </collision>
         <visual name="caster_back_visual">
-            <origin rpy="0 0 0" xyz="-0.08 0 -0.015"/>
+            <origin rpy="0 0 0" xyz="-0.08 0 -0.015" />
             <geometry>
-                <cylinder length="0.01" radius="0.003"/>
+                <cylinder length="0.01" radius="0.003" />
             </geometry>
         </visual>
     </link>
+    <joint name="dummy_joint" type="fixed">
+        <parent link="dummy" />
+        <child link="link_chassis" />
+        <origin rpy="0 0 0" xyz="0 0 0" />
+    </joint>
     <!-- simple line to indicate front -->
     <link name="front_indicator">
-        <parent link="link_chassis"/>
+        <parent link="link_chassis" />
         <visual>
-            <origin rpy="0 0 0" xyz="0.05 0 0"/>
+            <origin rpy="0 0 0" xyz="0.05 0 0" />
             <geometry>
-                <box size="0.045 0.005 0.001"/>
+                <box size="0.045 0.005 0.001" />
             </geometry>
         </visual>
     </link>
     <joint name="front_indicatior_joint" type="fixed">
-        <parent link="link_chassis"/>
-        <child link="front_indicator"/>
-        <origin rpy="0 0 0" xyz="0 0 0.071"/>
+        <parent link="link_chassis" />
+        <child link="front_indicator" />
+        <origin rpy="0 0 0" xyz="0 0 0.071" />
     </joint>
     <!-- <link name="sensor_laser">
@@ -129,7 +137,7 @@
     </joint> -->
     <!-- Create wheels -->
-    <xacro:link_wheel name="link_right_wheel"/>
-    <xacro:joint_wheel name="joint_right_wheel" child="link_right_wheel" origin_xyz="0 0.075 0"/>
-    <xacro:link_wheel name="link_left_wheel"/>
-    <xacro:joint_wheel name="joint_left_wheel" child="link_left_wheel" origin_xyz="0 -0.075 0"/>
+    <xacro:link_wheel name="link_right_wheel" />
+    <xacro:joint_wheel name="joint_right_wheel" child="link_right_wheel" origin_xyz="0 0.075 0" />
+    <xacro:link_wheel name="link_left_wheel" />
+    <xacro:joint_wheel name="joint_left_wheel" child="link_left_wheel" origin_xyz="0 -0.075 0" />
 </robot>

Commit message: feat: update launchfiles & rviz params

File: urdf/m2wr.xacro (robot description, xacro)
@@ -4,7 +4,4 @@
     <xacro:include filename="$(find mtracker)/urdf/m2wr.gazebo" />
     <xacro:include filename="$(find mtracker)/urdf/macro.xacro" />
-    <link name="dummy">
-        <pose>0 0 0 0 0 0</pose>
-    </link>
     <link name="link_chassis">
         <!-- pose and inertial -->
@@ -91,9 +88,4 @@
         </visual>
     </link>
-    <joint name="dummy_joint" type="fixed">
-        <parent link="dummy" />
-        <child link="link_chassis" />
-        <origin rpy="0 0 0" xyz="0 0 0" />
-    </joint>
     <!-- simple line to indicate front -->
     <link name="front_indicator">

Commit message: fix: fix intel nuc position

File: urdf/m2wr.xacro (robot description, xacro)
@@ -9,5 +9,5 @@
         <inertial>
             <mass value="1.8" />
-            <origin rpy="0 0 0" xyz="0 0 0.01" />
+            <origin xyz="0 0 0.01" />
             <inertia ixx="0.0395416666667" ixy="0" ixz="0" iyy="0.106208333333" iyz="0" izz="0.106208333333" />
         </inertial>
@@ -19,5 +19,5 @@
         </collision>
         <visual>
-            <origin rpy="0 0 0" xyz="0 0 0.010" />
+            <origin xyz="0 0 0.010" />
             <geometry>
                 <cylinder length="0.045" radius="0.084" />
@@ -27,5 +27,5 @@
         <!-- controller -->
         <visual>
-            <origin rpy="0 0 0" xyz="0 0 0.046" />
+            <origin xyz="0 0 0.045" />
             <geometry>
                 <cylinder length="0.025" radius="0.080" />
@@ -35,5 +35,5 @@
         <!-- intel nuc -->
         <visual>
-            <origin rpy="0 0 0" xyz="0 0 0.071" />
+            <origin xyz="0 0 0.087" />
             <geometry>
                 <box size="0.1 0.1 0.06" />

Commit message: feat: restore laser & fix its position and joint

File: urdf/m2wr.xacro (robot description, xacro)
@@ -103,19 +103,20 @@
         <origin rpy="0 0 0" xyz="0 0 0.071" />
     </joint>
-    <!-- <link name="sensor_laser">
+    <!-- Laser  -->
+    <link name="sensor_laser">
         <inertial>
-            <origin xyz="0 0 0" rpy="0 0 0"/>
+            <origin xyz="0 0 0"/>
             <mass value="0.1" />
             <xacro:cylinder_inertia mass="0.1" r="0.05" l="0.1" />
         </inertial>
         <visual>
-            <origin xyz="0 0 0" rpy="0 0 0"/>
+            <origin xyz="0 0 0" />
             <geometry>
-                <cylinder radius="0.05" length="0.1"/>
+                <cylinder radius="0.025" length="0.015"/>
             </geometry>
             <material name="white" />
         </visual>
         <collision>
-            <origin xyz="0 0 0" rpy="0 0 0"/>
+            <origin xyz="0 0 0"/>
             <geometry>
                 <cylinder radius="0.05" length="0.1"/>
@@ -124,8 +125,8 @@
     </link>
     <joint name="joint_sensor_laser" type="fixed">
-        <origin xyz="0.15 0 0.05" rpy="0 0 0"/>
+        <origin xyz="0 0 0.1245" />
         <parent link="link_chassis"/>
         <child link="sensor_laser"/>
-    </joint> -->
+    </joint>
     <!-- Create wheels -->
     <xacro:link_wheel name="link_right_wheel" />

File: urdf/macro.xacro (robot description, xacro)
@@ -34,8 +34,8 @@
     </xacro:macro>
     <!-- Laser scanner -->
-    <!-- <xacro:macro name="cylinder_inertia" params="mass r l">
+    <xacro:macro name="cylinder_inertia" params="mass r l">
       <inertia ixx="${mass*(3*r*r+l*l)/12}" ixy = "0" ixz = "0"
                iyy="${mass*(3*r*r+l*l)/12}" iyz = "0"
                izz="${mass*(r*r)/2}"/>
-    </xacro:macro> -->
+    </xacro:macro>
 </robot>

Commit message: fix: rename link_chassis to base_link

File: urdf/m2wr.xacro (robot description, xacro)
@@ -4,5 +4,5 @@
     <xacro:include filename="$(find mtracker)/urdf/m2wr.gazebo" />
     <xacro:include filename="$(find mtracker)/urdf/macro.xacro" />
-    <link name="link_chassis">
+    <link name="base_link">
         <!-- pose and inertial -->
         <pose>0 0 0.01 0 0 0</pose>
@@ -90,5 +90,5 @@
     <!-- simple line to indicate front -->
     <link name="front_indicator">
-        <parent link="link_chassis" />
+        <parent link="base_link" />
         <visual>
             <origin rpy="0 0 0" xyz="0.05 0 0" />
@@ -99,5 +99,5 @@
     </link>
     <joint name="front_indicatior_joint" type="fixed">
-        <parent link="link_chassis" />
+        <parent link="base_link" />
         <child link="front_indicator" />
         <origin rpy="0 0 0" xyz="0 0 0.071" />
@@ -126,5 +126,5 @@
     <joint name="joint_sensor_laser" type="fixed">
         <origin xyz="0 0 0.1245" />
-        <parent link="link_chassis"/>
+        <parent link="base_link"/>
         <child link="sensor_laser"/>
     </joint>

File: urdf/macro.xacro (robot description, xacro)
@@ -26,5 +26,5 @@
         <origin rpy="0 0 0" xyz="${origin_xyz}"/>
         <child link="${child}"/>
-        <parent link="link_chassis"/>
+        <parent link="base_link"/>
         <!-- <axis rpy="0 0 0" xyz="0 1 0"/> -->
         <axis xyz="0 1 0"/>
