Commit message: fix: odometry data now allows to build good maps with gmapping
it turned out that all the time the odometry was sent wrong, probably
the configuration wasn't written well. temporarily switching to ros_gazebo
plugin

File: urdf/mtracker.xacro (robot description, xacro)
@@ -29,5 +29,5 @@
             <origin xyz="0 0 0.045" />
             <geometry>
-                <cylinder length="0.025" radius="0.080" />
+                <cylinder length="0.022" radius="0.080" />
             </geometry>
             <material name="blue" />
@@ -45,5 +45,5 @@
             <origin rpy="0 0 0" xyz="0.08 0 -0.015" />
             <geometry>
-                <cylinder length="0.01" radius="0.003" />
+                <cylinder length="0.0215" radius="0.003" />
             </geometry>
             <surface>
@@ -61,5 +61,5 @@
             <origin rpy="0 0 0" xyz="0.08 0 -0.015" />
             <geometry>
-                <cylinder length="0.01" radius="0.003" />
+                <cylinder length="0.0215" radius="0.003" />
             </geometry>
         </visual>
@@ -68,5 +68,5 @@
             <origin rpy="0 0 0" xyz="-0.08 0 -0.015" />
             <geometry>
-                <cylinder length="0.01" radius="0.003" />
+                <cylinder length="0.0215" radius="0.003" />
             </geometry>
             <surface>
@@ -84,5 +84,5 @@
             <origin rpy="0 0 0" xyz="-0.08 0 -0.015" />
             <geometry>
-                <cylinder length="0.01" radius="0.003" />
+                <cylinder length="0.0215" radius="0.003" />
             </geometry>
         </visual>
